File: kicad/multical/multical.kicad_pcb (KiCad board)
At the start: 2 copper layers, 200 x 300 mm, 55 parts, among them J10 Screw_Terminal_01x02, J11 Screw_Terminal_01x02, J12 Screw_Terminal_01x02, J13 Screw_Terminal_01x02, J14 Screw_Terminal_01x02, J15 Screw_Terminal_01x02, J16 Screw_Terminal_01x02, J17 Screw_Terminal_01x02, J18 Screw_Terminal_01x02, K1 Relay_SPDT, K2 Relay_SPDT, K3 Relay_SPDT, K4 Relay_SPDT, K5 Relay_SPDT, K6 Relay_SPDT, K7 Relay_SPDT, K8 Relay_SPDT, U1 ESP32-WROOM-32, U10 HLK-PM01, U11 AMS1117-3.3, U12 zmpt101b, U13 ULN2003A, U14 ULN2003A, U2 ACS712xLCTR-20A, U3 ACS712xLCTR-20A, U4 ACS712xLCTR-20A, U5 ACS712xLCTR-20A, U6 ACS712xLCTR-20A, U7 ACS712xLCTR-20A, U8 ACS712xLCTR-20A, U9 ACS712xLCTR-20A

Commit message: Routage PCB 20A, schema de branchement et mise a jour de la presentation
- kicad/ : outils et guide de routage pour tenir 20A (GUIDE_ROUTAGE_20A,
  fix_dsn_widths_20A.py, replan_pcb_20A.py, strip_tracks.py), PCB/schema
  mis a jour en consequence. Routage non termine : il reste 10 pistes a
  tracer (cf. README racine).
- schema_branchement.png et diagramme_cas_utilisation.drawio ajoutes
- presentation de soutenance et GUIDE_MAQUETTE_BOITIER mis a jour
- retire l'ancienne sauvegarde du rapport (avant corrections)

Co-Authored-By: Claude Sonnet 5 <noreply@anthropic.com>
Other:
- board size 200 x 300 mm -> 236 x 461.5 mm
Changed lines of the file:
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@@
 	)
 	(setup
+		(stackup
+			(layer "F.Cu" (type "copper") (thickness 0.07))
+			(layer "dielectric 1" (type "core") (thickness 1.46) (material "FR4") (epsilon_r 4.5) (loss_tangent 0.02))
+			(layer "B.Cu" (type "copper") (thickness 0.07))
+			(copper_finish "None")
+			(dielectric_constraints no)
+		)
 		(pad_to_mask_clearance 0)
 		(allow_soldermask_bridges_in_footprints no)
@@
 	(gr_rect
 		(start 14 18.5)
-		(end 214 318.5)
+		(end 250 480)
 		(stroke
 			(width 0.05)
